Commit message: distill_kelun

File: legged_gym/resources/robots/g1_description/g1.urdf (robot description, URDF)
Before this commit: robot g1_29dof_with_hand_rev_1_0, 59 links, 58 joints
Joints:
- joint left_elbow_joint: axis 0 1 0 -> (none); limit lower=-1.0472 upper=2.0944 effort=25 velocity=37 -> (none); type revolute -> fixed
- joint left_shoulder_pitch_joint: axis 0 1 0 -> (none); limit lower=-3.0892 upper=2.6704 effort=25 velocity=37 -> (none); type revolute -> fixed
- joint left_shoulder_roll_joint: axis 1 0 0 -> (none); limit lower=-1.5882 upper=2.2515 effort=25 velocity=37 -> (none); type revolute -> fixed
- joint left_shoulder_yaw_joint: axis 0 0 1 -> (none); limit lower=-2.618 upper=2.618 effort=25 velocity=37 -> (none); type revolute -> fixed
- joint left_wrist_pitch_joint: axis 0 1 0 -> (none); limit lower=-1.614429558 upper=1.614429558 effort=5 velocity=22 -> (none); type revolute -> fixed
- joint left_wrist_roll_joint: axis 1 0 0 -> (none); limit lower=-1.972222054 upper=1.972222054 effort=25 velocity=37 -> (none); type revolute -> fixed
- joint left_wrist_yaw_joint: axis 0 0 1 -> (none); limit lower=-1.614429558 upper=1.614429558 effort=5 velocity=22 -> (none); type revolute -> fixed
- joint right_elbow_joint: axis 0 1 0 -> (none); limit lower=-1.0472 upper=2.0944 effort=25 velocity=37 -> (none); type revolute -> fixed
- joint right_shoulder_pitch_joint: axis 0 1 0 -> (none); limit lower=-3.0892 upper=2.6704 effort=25 velocity=37 -> (none); type revolute -> fixed
- joint right_shoulder_roll_joint: axis 1 0 0 -> (none); limit lower=-2.2515 upper=1.5882 effort=25 velocity=37 -> (none); type revolute -> fixed
- joint right_shoulder_yaw_joint: axis 0 0 1 -> (none); limit lower=-2.618 upper=2.618 effort=25 velocity=37 -> (none); type revolute -> fixed
- joint right_wrist_pitch_joint: axis 0 1 0 -> (none); limit lower=-1.614429558 upper=1.614429558 effort=5 velocity=22 -> (none); type revolute -> fixed
- joint right_wrist_roll_joint: axis 1 0 0 -> (none); limit lower=-1.972222054 upper=1.972222054 effort=25 velocity=37 -> (none); type revolute -> fixed
- joint right_wrist_yaw_joint: axis 0 0 1 -> (none); limit lower=-1.614429558 upper=1.614429558 effort=5 velocity=22 -> (none); type revolute -> fixed
- joint waist_yaw_joint: axis 0 0 1 -> (none); limit lower=-0.6 upper=0.6 effort=88 velocity=32 -> (none); type revolute -> fixed
